File: VixenBoard/SerialBoardVixen/SerialBoardVixen.kicad_sch (KiCad schematic)
At the start: 68 parts, among them J1 Jack-DC, J2 Connector, USB-TYPE-C-16P, J4 Conn_01x04_Pin, K1 RT44xxxx, K2 RT44xxxx, K3 RT44xxxx, K4 RT44xxxx, K5 RT44xxxx, K6 RT44xxxx, K7 RT44xxxx, K8 RT44xxxx, Q10 BC847, Q3 BC847, Q4 BC847, Q5 BC847, Q6 BC847, Q7 BC847, Q8 BC847, Q9 BC847, U1 AMS1117-3.3, U2 STM32F103C8T6, X1 X50328MSB2GI

Commit message: [UPD] Update electrical scheme
Parts:
- removed J2: Connector, USB-TYPE-C-16P, PCM_JLCPCB:TYPE-C-SMD_HX-TYPE-C-16PIN, symbol PCM_JLCPCB-Extended:Connector, USB-TYPE-C-16P
- added J2: USB_B, Connector_USB:USB_B_Lumberg_2411_02_Horizontal, symbol Connector:USB_B
- R1, R10, R15, R2, R3, R6, R7, R8, R9: value 220 -> 330
Connections:
- net GND: now also J2.4 (GND)
- net VBUS: now also J2.1 (VBUS)
- net at R14.2: now also J2.2 (D-)
- net at R13.2: now also J2.3 (D+)
- no-connect marks 19 -> 16
